File: design/pcb/frida65A.kicad_sch (KiCad schematic)
At the start: 101 parts, among them J1 DisplayPort Molex 472720024, J10 VIN CFG, J11 TP AMP, J12 MiniFitJr Molex 469990014, J13 POWER, J14 RJ45 Molex 446200002, J15 SPI TP, J2 TP CLOCKS, J3 SMA Molex 733910070, J4 SMA Molex 733910070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

Commit message: chore(pcb): update schematic and layout
Parts:
- removed Q1: Q_PMOS_DGS, Package_TO_SOT_SMD:SOT-23-3, symbol Transistor_FET:Q_PMOS_DGS
- added Q1: Q_PMOS_GSD, Package_TO_SOT_SMD:SOT-23, symbol Transistor_FET:Q_PMOS_GSD
Connections:
- net AMP_PD_EXT: now also Q1.1 (G)
- net AMP_PD_N: now also Q1.3 (D)
- net VDD_BDAQ: now also Q1.2 (S)
Other:
- note added: "VDD_BDAQ should be 2.5V"
- note added: "VS_N should be -1V"
- note removed: "1.2V"
Changed lines of the file:
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@@
 		)
 	)
-	(text "1.2V"
+	(text "2.5V"
 		(exclude_from_sim no)
 		(at 203.2 182.88 0)
@@
 		)
 	)
+	(text "VDD_BDAQ should be 2.5V"
+		(exclude_from_sim no)
+		(at 160.02 156.21 0)
+		(effects
+			(font
+				(size 1.27 1.27)
+			)
+			(justify left)
+		)
+	)
 	(text "AMP\nON"
 		(exclude_from_sim no)
@@
 		)
 	)
+	(text "VS_N should be -1V\n"
+		(exclude_from_sim no)
+		(at 180.34 196.85 0)
+		(effects
+			(font
+				(size 1.27 1.27)
+			)
+			(justify left)
+		)
+	)
 	(text "AMP\nOFF"
 		(exclude_from_sim no)
@@
 	(wire
 		(pts
-			(xy 349.25 36.83) (xy 358.14 36.83)
+			(xy 354.33 36.83) (xy 358.14 36.83)
 		)
 		(stroke
@@
 	(wire
 		(pts
-			(xy 349.25 41.91) (xy 358.14 41.91)
+			(xy 354.33 41.91) (xy 358.14 41.91)
 		)
 		(stroke
@@
 	(wire
 		(pts
-			(xy 349.25 39.37) (xy 358.14 39.37)
+			(xy 354.33 39.37) (xy 358.14 39.37)
 		)
 		(stroke
@@
 	(wire
 		(pts
-			(xy 349.25 34.29) (xy 358.14 34.29)
+			(xy 354.33 34.29) (xy 358.14 34.29)
 		)
 		(stroke
@@
 	)
 	(label "VOCM_EXT"
-		(at 349.25 39.37 180)
+		(at 354.33 39.37 180)
 		(effects
 			(font
@@
 	)
 	(label "VIN_P_EXT"
-		(at 349.25 34.29 180)
+		(at 354.33 34.29 180)
 		(effects
 			(font
@@
 	)
 	(label "AMP_PD_EXT"
-		(at 349.25 41.91 180)
+		(at 354.33 41.91 180)
 		(effects
 			(font
@@
 	)
 	(label "VIN_N_EXT"
-		(at 349.25 36.83 180)
+		(at 354.33 36.83 180)
 		(effects
 			(font
@@
 	)
 	(symbol
-		(lib_id "Transistor_FET:Q_PMOS_DGS")
-		(at 176.53 173.99 0)
-		(mirror x)
-		(unit 1)
-		(exclude_from_sim no)
-		(in_bom yes)
-		(on_board yes)
-		(dnp no)
-		(property "Reference" "Q1"
-			(at 182.88 175.2601 0)
-			(effects
-				(font
-					(size 1.27 1.27)
-				)
-				(justify left)
-			)
-		)
-		(property "Value" "Q_PMOS_DGS"
-			(at 182.88 172.7201 0)
-			(effects
-				(font
-					(size 1.27 1.27)
-				)
-				(justify left)
-			)
-		)
-		(property "Footprint" "Package_TO_SOT_SMD:SOT-23-3"
-			(at 181.61 176.53 0)
-			(effects
-				(font
-					(size 1.27 1.27)
-				)
-				(hide yes)
-			)
-		)
-		(property "Datasheet" "~"
-			(at 176.53 173.99 0)
-			(effects
-				(font
-					(size 1.27 1.27)
-				)
-				(hide yes)
-			)
-		)
-		(property "Description" "P-MOSFET transistor, drain/gate/source"
-			(at 176.53 173.99 0)
-			(effects
-				(font
-					(size 1.27 1.27)
-				)
-				(hide yes)
-			)
-		)
-		(property "Sim.Device" ""
-			(at 176.53 173.99 0)
-			(effects
-				(font
-					(size 1.27 1.27)
-				)
-				(hide yes)
-			)
-		)
-		(property "Sim.Pins" ""
-			(at 176.53 173.99 0)
-			(effects
-				(font
-					(size 1.27 1.27)
-				)
-				(hide yes)
-			)
-		)
-		(property "Sim.Type" ""
-			(at 176.53 173.99 0)
-			(effects
-				(font
-					(size 1.27 1.27)
-				)
-				(hide yes)
-			)
-		)
-		(pin "1"
-		)
-		(pin "2"
-		)
-		(pin "3"
-		)
-		(instances
-			(project ""
-				(path "/fa3d0b93-951b-4460-b2d5-04f3ffae1154"
-					(reference "Q1")
-					(unit 1)
-				)
-			)
-		)
-	)
-	(symbol
 		(lib_id "Device:R")
 		(at 104.14 115.57 0)
@@
 					(unit 1)
 				)
+			)
+		)
+	)
+	(symbol
+		(lib_id "Transistor_FET:Q_PMOS_GSD")
+		(at 176.53 173.99 0)
+		(mirror x)
+		(unit 1)
+		(exclude_from_sim no)
+		(in_bom yes)
+		(on_board yes)
+		(dnp no)
+		(property "Reference" "Q1"
+			(at 182.88 175.2601 0)
+			(effects
+				(font
+					(size 1.27 1.27)
+				)
+				(justify left)
+			)
+		)
+		(property "Value" "Q_PMOS_GSD"
+			(at 182.88 172.7201 0)
+			(effects
+				(font
+					(size 1.27 1.27)
+				)
+				(justify left)
+			)
+		)
+		(property "Footprint" "Package_TO_SOT_SMD:SOT-23"
+			(at 181.61 176.53 0)
+			(effects
+				(font
+					(size 1.27 1.27)
+				)
+				(hide yes)
+			)
+		)
+		(property "Datasheet" "https://www.onsemi.com/pdf/datasheet/bss84-d.pdf"
+			(at 176.53 173.99 0)
+			(effects
+				(font
+					(size 1.27 1.27)
+				)
+				(hide yes)
+			)
+		)
+		(property "Description" "P-MOSFET transistor, gate/source/drain"
+			(at 176.53 173.99 0)
+			(effects
+				(font
+					(size 1.27 1.27)
+				)
+				(hide yes)
+			)
+		)
+		(pin "2"
+		)
+		(pin "3"
+		)
+		(pin "1"
+		)
+		(instances
+			(project "frida65A"
+				(path "/fa3d0b93-951b-4460-b2d5-04f3ffae1154"
+					(reference "Q1")
+					(unit 1)
+				)
