File: design/pcb/frida65A.kicad_pcb (KiCad board)
At the start: 4 copper layers, 100 x 100 mm, 105 parts, among them J1 DisplayPort Molex 472720024, J10 VIN CFG, J11 TP AMP, J12 MiniFitJr Molex 469990014, J13 POWER, J14 RJ45 Molex 446200002, J15 SPI TP, J2 TP CLOCKS, J3 SMA Molex 733910070, J4 SMA Molex 733910070, J5 DIFF/SE CFG, J6 TERM CFG, J7 ATTEN CFG, J8 SMA Molex 733910070, J9 TERM CFG, Q1 Q_PMOS_GSD, U1 DiffAmp TI THS4541, U2 TI LevelShifter SN74AXC8T245R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, U3 ASIC FRIDA 65A

Commit message: chore(pcb): update KiCad design files
Parts:
- Q1: value Q_PMOS_GSD -> (none)
- moved R31 0.72 mm to (158.8, 84.6)
- moved R32 0.72 mm to (156.9, 78.8)
- moved Q1 0.64 mm to (158.8, 82.0), turned to 90 degrees
Routing:
- net /AMP_PD_EXT: track 86.5 -> 77.4 mm, vias 4 -> 2
- net /AMP_PD_N: track 25.9 -> 23.1 mm
- net /VDD_BDAQ: track 111.4 -> 109.8 mm
- net /VIN_P: track 43.2 -> 44.5 mm
- net /VIN_N: track 36.5 -> 37.6 mm
